Commit message: -

File: urdf/example_robot.urdf.xacro (robot description, xacro)
@@ -2,14 +2,13 @@
 <robot xmlns:xacro="http://www.ros.org/wiki/xacro" name="robot">
     <xacro:include filename="example_include.xacro" />
-  <!-- ****************** ROBOT BASE FOOTPRINT ***************************  -->
-  <!-- Define the center of the main robot chassis projected on the ground -->
-  <link name="base_footprint"/>
-  <!-- ********************** ROBOT BASE *********************************  -->
-	<joint name="base_joint" type="fixed">
-	<origin xyz="0 0 0" rpy="0 0 0"/>
-	<parent link="base_footprint"/>
-	<child link="base_link"/>
-	</joint>
--
+    <!-- ****************** ROBOT BASE FOOTPRINT ***************************  -->
+    <!-- Define the center of the main robot chassis projected on the ground -->
+    <link name="base_footprint"/>
+    <!-- ********************** ROBOT BASE *********************************  -->
+    <joint name="base_joint" type="fixed">
+        <origin xyz="0 0 0" rpy="0 0 0"/>
+        <parent link="base_footprint"/>
+        <child link="base_link"/>
+    </joint>
     <link name="base_link">
         <visual>
@@ -32,9 +31,9 @@
         <parent link="base_link"/>
         <child link="lidar_link"/>
-        <origin xyz="0 0 0.2" rpy="0 0 0"/>
+        <origin xyz="0 0 0.4" rpy="0 0 0"/>
     </joint>
     <link name="lidar_link">
         <visual>
-            <origin xyz="0 0 0.25" rpy="0 0 0"/>
+            <origin xyz="0 0 0.4" rpy="0 0 0"/>
             <geometry>
                 <cylinder radius="0.05" length="0.16"/>

Commit message: urdf

File: urdf/example_robot.urdf.xacro (robot description, xacro)
@@ -7,5 +7,5 @@
     <!-- ********************** ROBOT BASE *********************************  -->
     <joint name="base_joint" type="fixed">
-        <origin xyz="0 0 0" rpy="0 0 0"/>
+        <origin xyz="0 0 0.04" rpy="0 0 0"/>
         <parent link="base_footprint"/>
         <child link="base_link"/>
@@ -15,8 +15,8 @@
             <origin xyz="0 0 0.00" rpy="0 0 0"/>
             <geometry>
-                <box size="0.35 0.35 0.2" />
+                <box size="0.23 0.25 0.08" />
             </geometry>
-            <material name="green">
-                <color rgba="0.2 1 0.2 1"/>
+            <material name="grey">
+                <color rgba=".2 .2 .2 1"/>
             </material>
         </visual>
@@ -24,5 +24,5 @@
             <origin xyz="0 0 0.00" rpy="0 0 0"/>
             <geometry>
-                <box size="0.4 0.4 0.25" />
+                <box size="0.30 0.30 0.08" />
             </geometry>
         </collision>
@@ -31,14 +31,14 @@
         <parent link="base_link"/>
         <child link="lidar_link"/>
-        <origin xyz="0 0 0.4" rpy="0 0 0"/>
+        <origin xyz="0.05 0 0.08" rpy="0 0 0"/>
     </joint>
     <link name="lidar_link">
         <visual>
-            <origin xyz="0 0 0.4" rpy="0 0 0"/>
+            <origin xyz="0 0 0" rpy="0 0 0"/>
             <geometry>
-                <cylinder radius="0.05" length="0.16"/>
+                <cylinder radius="0.05" length="0.08"/>
             </geometry>
-            <material name="green">
-                <color rgba="0.2 1 0.2 1"/>
+            <material name="Lgrey">
+                <color rgba=".5 .5 .5 1"/>
             </material>
         </visual>

Commit message: pre cleaup

File: urdf/example_robot.urdf.xacro (robot description, xacro)
@@ -30,8 +30,8 @@
     <joint name="lidar_joint" type="fixed">
         <parent link="base_link"/>
-        <child link="lidar_link"/>
+        <child link="laser"/>
         <origin xyz="0.05 0 0.08" rpy="0 0 0"/>
     </joint>
-    <link name="lidar_link">
+    <link name="laser">
         <visual>
             <origin xyz="0 0 0" rpy="0 0 0"/>
